File: onekeyboard_1/onekeyboard_1.brd (EAGLE design)
At the start: 28 x 28 mm, 21 parts, among them IC1 MCP1703AT, J2 CORTEX_DEBUG_PTH, U1 ATSAMD21G-A, X2 ZX62D-B-5PA8, Y1 32.768kHz

Commit message: sent to fab
Parts:
- removed H1, H2: MOUNT-HOLE2.8, holes:2,8
- added Q1: 220mA/50V/3.5Ω, SparkFun-DiscreteSemi:SOT23-3
- added R_MOSFET: (no value), SparkFun-Passives:0805
- moved RRST1 8.71 mm to (12.3, 2.50), turned to 270 degrees
- moved R_LED 5.64 mm to (12.6, 5.00), flipped to the top, turned to 0 degrees
- moved C4 4.18 mm to (22.4, 1.38)
- moved C5 3.24 mm to (26.6, 8.00), turned to 270 degrees
- moved Y1 1.55 mm to (23.2, 5.40)
- moved TP3 1.22 mm to (26.0, 23.6)
- moved TP1 1.00 mm to (21.0, 26.0)
- moved TP2 1.00 mm to (24.0, 26.0)
- moved C25 0.45 mm to (14.0, 5.40)
- moved C9 0.13 mm to (26.6, 4.60)
- flipped J2 to the top, turned to 270 degrees
Connections:
- removed net BTN: U1.47
- removed net CAM1: U1.23
- removed net CAM2: U1.24
- removed net USB0_EN: U1.26
- removed net USB1_EN: U1.30
- removed net USB2_EN: U1.28
- new net N$1: Q1.2, R_LED.2
- new net N$2: Q1.1, R_MOSFET.1
- net BUTTON: now also U1.27
- net GND: now also S1.K; no longer R_LED.2
- net LED: now also R_MOSFET.2, U1.47; no longer S1.K, U1.27
- net VCC: now also Q1.3
Routing:
- net VCC: track 22.2 -> 84.8 mm, vias 12 -> 13
- net LED: track 0.00 -> 47.1 mm, vias 0 -> 1
- net BUTTON: track 0.00 -> 26.7 mm, vias 0 -> 1
- net RX: track 0.00 -> 24.3 mm, vias 0 -> 2
- net TX: track 0.00 -> 21.9 mm, vias 0 -> 2
- net GND: track 10.3 -> 25.8 mm, vias 7 -> 14
- net RESET: track 24.4 -> 16.7 mm, vias 0 -> 1
- net N$4: track 0.00 -> 4.76 mm
- net N$2: track 0.00 -> 2.02 mm
- net N$1: track 0.00 -> 1.69 mm
- net SWDIO: track 15.9 -> 14.9 mm, vias 1 -> 0
- net N$32: track 7.92 -> 8.75 mm
- net SWDCLK: track 15.2 -> 14.6 mm
Other:
- outline, holes or cut-outs redrawn
- board text added: "A"
- board text added: "GND"
- board text added: "OKB"
- board text added: "RX"
- board text added: "TX"
- board text added: "rev."
