File: onekeyboard_1/onekeyboard_1.sch (EAGLE design)
At the start: 21 parts, among them IC1 MCP1703AT, J2 CORTEX_DEBUG_PTH, U1 ATSAMD21G-A, X2 ZX62D-B-5PA8, Y1 32.768kHz

Commit message: sent to fab
Parts:
- removed H1, H2: MOUNT-HOLE2.8, holes:MOUNT-HOLE2.8
- added Q1: 220mA/50V/3.5Ω, SparkFun-DiscreteSemi:MOSFET-NCH-BSS138
- added R_MOSFET: (no value), SparkFun-Passives:RESISTOR0805-RES
Connections:
- removed net BTN: U1.PB02(AIN10/SER5:0)
- removed net CAM1: U1.PA14(XIN/SER2:2+)
- removed net CAM2: U1.PA15(XOUT/SER2:3+)
- removed net USB0_EN: U1.PA17(I2C/SER1:1+)
- removed net USB1_EN: U1.PA21(SER5:3+)
- removed net USB2_EN: U1.PA19(SER1:3+)
- new net N$1: Q1.S, R_LED.2
- new net N$2: Q1.G, R_MOSFET.1
- net BUTTON: now also U1.PA18(SER1:2+)
- net GND: now also S1.C; no longer R_LED.2
- net LED: now also R_MOSFET.2, U1.PB02(AIN10/SER5:0); no longer S1.C, U1.PA18(SER1:2+)
- net VCC: now also Q1.D
