File: onekeyboard_2/onekeyboard_2.brd (EAGLE design)
At the start: 28 x 28 mm, 21 parts, among them IC1 MCP1703AT, J2 CORTEX_DEBUG_PTH, Q1 220mA/50V/3.5Ω, U1 ATSAMD21G-A, X2 ZX62D-B-5PA8, Y1 32.768kHz

Commit message: rev B eagle files
Parts:
- moved R_MOSFET 3.41 mm to (12.2, 2.20), turned to 270 degrees
- moved Q1 3.16 mm to (15.2, 4.20), turned to 0 degrees
- moved R_LED 1.41 mm to (11.2, 4.80), turned to 180 degrees
- moved C1 0.10 mm to (15.0, 3.70)
Connections:
- removed net CAM_EN: U1.10
- removed net N$1 (its old number): Q1.2, R_LED.2
- removed net VD_INT: U1.7
- new net N$3: Q1.3, S1.K
- net GND: now also Q1.2; no longer S1.K
- net VCC: now also R_LED.2; no longer Q1.3
Routing:
- net N$3: track 0.00 -> 3.65 mm
- net LED: track 47.1 -> 48.9 mm
- net N$1 (its old number): track 1.69 -> 0.00 mm
- net VCC: track 84.8 -> 83.4 mm
Other:
- board text added: "B"
- board text removed: "A"
