File: onekeyboard_2/onekeyboard_2.sch (EAGLE design)
At the start: 21 parts, among them IC1 MCP1703AT, J2 CORTEX_DEBUG_PTH, Q1 220mA/50V/3.5Ω, U1 ATSAMD21G-A, X2 ZX62D-B-5PA8, Y1 32.768kHz

Commit message: rev B eagle files
Connections:
- removed net CAM_EN: U1.PA05(AIN5/SER0:1/TC0:1)
- removed net N$1 (its old number): Q1.S, R_LED.2
- removed net VD_INT: U1.PB08(AIN2/SER4:0/TC4:0)
- new net N$3: Q1.D, S1.C
- net GND: now also Q1.S; no longer S1.C
- net VCC: now also R_LED.2; no longer Q1.D
